File: Analog2HDMI.kicad_pcb (KiCad board)
At the start: 2 copper layers, 100 x 48.5 mm, 18 parts, among them J1 USB_C_Receptacle_USB2.0, J10 Conn_01x01, J2 DB15_Female_HighDensity_Mount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, J3 Conn_Coaxial, J4 Conn_Coaxial, J5 Conn_Coaxial, J6 Conn_Coaxial, J7 Conn_Coaxial, J8 Conn_Coaxial, J9 Conn_01x01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

Commit message: updated to latest version
Parts:
- added C1: 220u, Capacitor_SMD:C_1206_3216Metric_Pad1.33x1.80mm_HandSolder, F.Cu at (170.1, 78.8)
- added C2: C_Polarized, Capacitor_SMD:CP_Elec_6.3x7.7, F.Cu at (169.9, 80.7)
- added R2: 5k1, Resistor_SMD:R_1206_3216Metric, F.Cu at (111.7, 62.2)
- added REF**: Circuit-Board-Logo, Eigene:Circuit-Board-Logo, B.Cu at (124.1, 59.9)
- J3: footprint Connector_Coaxial:RCA_Green -> Connector_Coaxial:AV-8.4-9
- J4: footprint Connector_Coaxial:RCA_Blue -> Connector_Coaxial:AV-8.4-9
- J5, J6: footprint Connector_Coaxial:RCA_Red -> Connector_Coaxial:AV-8.4-9
- J7: footprint Connector_Coaxial:RCA_White -> Connector_Coaxial:AV-8.4-9
- J8: footprint Connector_Coaxial:RCA_Gray -> Connector_Coaxial:AV-8.4-9
- moved J4 4.29 mm to (166.2, 96.0)
- moved J3 4.28 mm to (152.2, 96.0)
- moved J5 4.28 mm to (180.2, 96.0)
- moved J2 2.93 mm to (131.1, 92.5)
- moved R1 2.55 mm to (111.7, 59.2), turned to 180 degrees
- moved J7 1.60 mm to (196.0, 89.8)
- moved J8 1.60 mm to (196.0, 61.8)
- moved J6 1.59 mm to (196.0, 75.8)
- moved J9 1.11 mm to (138.7, 69.5)
- moved H4 1.08 mm to (184.7, 84.0)
- moved U1 1.04 mm to (150.0, 68.0)
- moved J10 0.84 mm to (161.3, 67.2)
Connections:
- net /~ANALOG renamed /~{ANALOG}
- net /~RGBHV renamed /~{RGBHV}
- J1 pad A6: (no net) -> unconnected-(J1-PadA6)
- J1 pad A7: (no net) -> unconnected-(J1-PadA7)
- J1 pad A8: (no net) -> unconnected-(J1-PadA8)
- J1 pad B5: Net-(J1-PadA5) -> Net-(J1-PadB5)
- J1 pad B6: (no net) -> unconnected-(J1-PadB6)
- J1 pad B7: (no net) -> unconnected-(J1-PadB7)
- J1 pad B8: (no net) -> unconnected-(J1-PadB8)
- J2 pad 0: Net-(J2-Pad0) -> unconnected-(J2-Pad0)
- J2 pad 11: (no net) -> unconnected-(J2-Pad11)
- J2 pad 12: (no net) -> unconnected-(J2-Pad12)
- J2 pad 15: (no net) -> unconnected-(J2-Pad15)
- J2 pad 4: (no net) -> unconnected-(J2-Pad4)
- SW1 pad 1: (no net) -> unconnected-(SW1-Pad1)
- SW2 pad 1: (no net) -> unconnected-(SW2-Pad1)
Routing:
- net /G|Y: track 48.6 -> 36.4 mm
- net /SPDIF: track 73.1 -> 60.9 mm
- net /B|Pb: track 65.8 -> 54.2 mm
- net +5V: track 93.1 -> 104.5 mm
- net /R|Pr: track 72.2 -> 62.8 mm
- net Net-(J1-PadA5): track 9.45 -> 3.15 mm
- net /VS: track 39.0 -> 45.0 mm
- net /HS: track 32.7 -> 38.6 mm
- net GND: track 4.26 -> 0.03 mm, vias 0 -> 1
- net Net-(J1-PadB5): track 0.00 -> 3.15 mm
- net /AUDIO_R: track 57.0 -> 54.8 mm
- net /~{RGBHV}: track 37.8 -> 38.8 mm
- net /~{ANALOG}: track 76.7 -> 77.6 mm
Other:
- outline, holes or cut-outs redrawn
- net class Default removed
- net class Supply removed
- board text added: "Analog2HDMI Carrier-Board By ManCloud v20220319"
- board text added: "Powered by: - jotheripper - derKevin - FuNzeL - BambooShadow"
- board text removed: "Analog2HDMI Carrier-Board By ManCloud v20211213"
